File: pcb/pcb.kicad_pcb (KiCad board)
At the start: 2 copper layers, 74 x 47 mm, 11 parts, among them SW1 generate, SW2 down, SW3 up, SW4 power sw, U1 MOUDLE-SEEEDUINO-XIAO

Commit message: thing
Parts:
- removed G***: LOGO, LOGO
- removed SW4: power sw, Button_Switch_THT:SW_Slide_SPDT_Straight_CK_OS102011MS2Q
- removed adafruitbq1: ~, adafruit bq25185:adafruit bq25185
- added H3: MountingHole_Pad, MountingHole:MountingHole_3.2mm_M3_Pad_Via, F.Cu at (111.5, 98.0)
- added J1: Conn_01x02_Pin, Connector_PinHeader_1.00mm:PinHeader_1x02_P1.00mm_Vertical, F.Cu at (128.5, 95.6)
- U1: value MOUDLE-SEEEDUINO-XIAO -> XIAO-RP2350-SMD-MODEL; footprint seed studio xiao:MOUDLE14P-2.54-21X17.8MM -> seed studio xiao:XIAO-RP2350-SMD-MODEL
- moved H1 31.7 mm to (111.5, 135.0)
- moved U1 23.2 mm to (117.2, 118.7), turned to 180 degrees
- moved SW1 1.77 mm to (117.0, 133.0)
- moved SSD1306 1.75 mm to (106.6, 102.1)
- moved SW2 1.75 mm to (137.7, 121.2)
- moved SW3 1.75 mm to (137.7, 108.5)
- moved H4 0.07 mm to (143.8, 98.0)
Connections:
- net Net-(SSD1306-VCC) renamed +3V3
- U1 pad 14: Net-(U1-5V) -> unconnected-(U1-VBUS-Pad14)
- U1 pad 4: unconnected-(U1-PA11_A3_D3-Pad4) -> Net-(SSD1306-SDA)
- U1 pad 5: Net-(SSD1306-SDA) -> Net-(SSD1306-SCL)
- U1 pad 6: Net-(SSD1306-SCL) -> unconnected-(U1-D5-Pad6)
Routing:
- net +3V3: track 39.8 -> 7.63 mm
- net Net-(U1-5V): track 30.4 -> 0.00 mm
- net Net-(J1-Pin_1): track 0.00 -> 28.0 mm, vias 0 -> 1
- net Net-(J1-Pin_2): track 0.00 -> 23.7 mm
- net Net-(adafruitbq1-EN): track 21.3 -> 0.00 mm
- net Net-(U1-D1): track 44.4 -> 36.4 mm
- net Net-(U1-D0): track 20.4 -> 26.5 mm
- net Net-(SSD1306-SDA): track 31.2 -> 25.8 mm, vias 0 -> 2
- net Net-(U1-D2): track 48.6 -> 43.5 mm
- net Net-(SSD1306-SCL): track 27.6 -> 23.8 mm
Other:
- board size 74 x 47 mm -> 42.2 x 47 mm
- board text added: "+"
- board text added: "-"
- board text added: "KO6LBA V0.2"
- board text removed: "KO6LBA V0.1"
