File: pcb/_restore_backup_2026-08-02T03-03-27-170/pcb.kicad_sch (KiCad schematic)
At the start: 10 parts, among them J1 Conn_01x02_Pin, SW1 generate, SW2 down, SW3 up, U1 XIAO-RP2350-SMD-MODEL

Commit message: thing
Parts:
- removed J1: Conn_01x02_Pin, Connector_PinHeader_1.00mm:PinHeader_1x02_P1.00mm_Vertical, symbol Connector:Conn_01x02_Pin
- U1: value XIAO-RP2350-SMD-MODEL -> XIAO-RP2350-SMD; footprint seed studio xiao:XIAO-RP2350-SMD-MODEL -> Seeed_Studio_XIAO_Series:XIAO-RP2350-SMD
Connections:
- net GND: no longer U1.26 (GND)
- no-connect marks 20 -> 23
Changed lines of the file:
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@@
 	(text_box "pin map"
 		(exclude_from_sim no)
-		(at 163.83 137.16 0)
+		(at 153.67 146.05 0)
 		(size 12.7 2.54)
 		(margins 0.9525 0.9525 0.9525 0.9525)
@@
 	)
 	(no_connect
+		(at 137.16 78.74)
+	)
+	(no_connect
 		(at 158.75 97.79)
 	)
@@
 	)
 	(no_connect
+		(at 133.35 130.81)
+	)
+	(no_connect
 		(at 158.75 105.41)
 	)
@@
 	)
 	(no_connect
+		(at 137.16 130.81)
+	)
+	(no_connect
 		(at 158.75 121.92)
 	)
@@
 	(wire
 		(pts
-			(xy 133.35 130.81) (xy 133.35 137.16)
-		)
-		(stroke
-			(width 0)
-			(type default)
-		)
-	)
-	(wire
-		(pts
 			(xy 107.95 97.79) (xy 113.03 97.79)
 		)
@@
 	(wire
 		(pts
-			(xy 137.16 137.16) (xy 135.89 137.16)
-		)
-		(stroke
-			(width 0)
-			(type default)
-		)
-	)
-	(wire
-		(pts
 			(xy 102.87 101.6) (xy 102.87 128.27)
 		)
@@
 		(pts
 			(xy 198.12 110.49) (xy 198.12 115.57)
-		)
-		(stroke
-			(width 0)
-			(type default)
-		)
-	)
-	(wire
-		(pts
-			(xy 137.16 130.81) (xy 137.16 137.16)
 		)
 		(stroke
@@
 			(table_cell "d0"
 				(exclude_from_sim no)
-				(at 163.83 139.7 0)
+				(at 153.67 148.59 0)
 				(size 3.81 2.54)
 				(margins 0.9525 0.9525 0.9525 0.9525)
@@
 			(table_cell "GPIO26"
 				(exclude_from_sim no)
-				(at 167.64 139.7 0)
+				(at 157.48 148.59 0)
 				(size 8.89 2.54)
 				(margins 0.9525 0.9525 0.9525 0.9525)
@@
 			(table_cell "d1"
 				(exclude_from_sim no)
-				(at 163.83 142.24 0)
+				(at 153.67 151.13 0)
 				(size 3.81 2.54)
 				(margins 0.9525 0.9525 0.9525 0.9525)
@@
 			(table_cell "GPIO27"
 				(exclude_from_sim no)
-				(at 167.64 142.24 0)
+				(at 157.48 151.13 0)
 				(size 8.89 2.54)
 				(margins 0.9525 0.9525 0.9525 0.9525)
@@
 			(table_cell "d2"
 				(exclude_from_sim no)
-				(at 163.83 144.78 0)
+				(at 153.67 153.67 0)
 				(size 3.81 2.54)
 				(margins 0.9525 0.9525 0.9525 0.9525)
@@
 			(table_cell "GPIO28"
 				(exclude_from_sim no)
-				(at 167.64 144.78 0)
+				(at 157.48 153.67 0)
 				(size 8.89 2.54)
 				(margins 0.9525 0.9525 0.9525 0.9525)
@@
 			(table_cell "d4"
 				(exclude_from_sim no)
-				(at 163.83 147.32 0)
+				(at 153.67 156.21 0)
 				(size 3.81 2.54)
 				(margins 0.9525 0.9525 0.9525 0.9525)
@@
 			(table_cell "GPIO6"
 				(exclude_from_sim no)
-				(at 167.64 147.32 0)
+				(at 157.48 156.21 0)
 				(size 8.89 2.54)
 				(margins 0.9525 0.9525 0.9525 0.9525)
@@
 			(table_cell "d5"
 				(exclude_from_sim no)
-				(at 163.83 149.86 0)
+				(at 153.67 158.75 0)
 				(size 3.81 2.54)
 				(margins 0.9525 0.9525 0.9525 0.9525)
@@
 			(table_cell "GPIO7"
 				(exclude_from_sim no)
-				(at 167.64 149.86 0)
+				(at 157.48 158.75 0)
 				(size 8.89 2.54)
 				(margins 0.9525 0.9525 0.9525 0.9525)
@@
 					)
 					(justify left top)
-				)
-			)
-		)
-	)
-	(symbol
-		(lib_id "power:GND")
-		(at 137.16 78.74 180)
-		(unit 1)
-		(body_style 1)
-		(exclude_from_sim no)
-		(in_bom yes)
-		(on_board yes)
-		(in_pos_files yes)
-		(dnp no)
-		(fields_autoplaced yes)
-		(property "Reference" "#PWR010"
-			(at 137.16 72.39 0)
-			(hide yes)
-			(show_name no)
-			(do_not_autoplace no)
-			(effects
-				(font
-					(size 1.27 1.27)
-				)
-			)
-		)
-		(property "Value" "GND"
-			(at 137.16 73.66 0)
-			(show_name no)
-			(do_not_autoplace no)
-			(effects
-				(font
-					(size 1.27 1.27)
-				)
-			)
-		)
-		(property "Footprint" ""
-			(at 137.16 78.74 0)
-			(hide yes)
-			(show_name no)
-			(do_not_autoplace no)
-			(effects
-				(font
-					(size 1.27 1.27)
-				)
-			)
-		)
-		(property "Datasheet" ""
-			(at 137.16 78.74 0)
-			(hide yes)
-			(show_name no)
-			(do_not_autoplace no)
-			(effects
-				(font
-					(size 1.27 1.27)
-				)
-			)
-		)
-		(property "Description" "Power symbol creates a global label with name \"GND\" , ground"
-			(at 137.16 78.74 0)
-			(hide yes)
-			(show_name no)
-			(do_not_autoplace no)
-			(effects
-				(font
-					(size 1.27 1.27)
-				)
-			)
-		)
-		(pin "1"
-		)
-		(instances
-			(project "pcb"
-				(path "/bb6da232-368e-4a1f-bf9d-dbd7b03483b8"
-					(reference "#PWR010")
-					(unit 1)
 				)
 			)
@@
 	)
 	(symbol
-		(lib_id "Connector:Conn_01x02_Pin")
-		(at 133.35 142.24 90)
-		(unit 1)
-		(body_style 1)
-		(exclude_from_sim no)
-		(in_bom yes)
-		(on_board yes)
-		(in_pos_files yes)
-		(dnp no)
-		(fields_autoplaced yes)
-		(property "Reference" "J1"
-			(at 137.16 140.3349 90)
-			(show_name no)
-			(do_not_autoplace no)
-			(effects
-				(font
-					(size 1.27 1.27)
-				)
-				(justify right)
-			)
-		)
-		(property "Value" "Conn_01x02_Pin"
-			(at 137.16 142.8749 90)
-			(show_name no)
-			(do_not_autoplace no)
-			(effects
-				(font
-					(size 1.27 1.27)
-				)
-				(justify right)
-			)
-		)
-		(property "Footprint" "Connector_PinHeader_1.00mm:PinHeader_1x02_P1.00mm_Vertical"
-			(at 133.35 142.24 0)
-			(hide yes)
-			(show_name no)
-			(do_not_autoplace no)
-			(effects
-				(font
-					(size 1.27 1.27)
-				)
-			)
-		)
-		(property "Datasheet" ""
-			(at 133.35 142.24 0)
-			(hide yes)
-			(show_name no)
-			(do_not_autoplace no)
-			(effects
-				(font
-					(size 1.27 1.27)
-				)
-			)
-		)
-		(property "Description" "Generic connector, single row, 01x02, script generated"
-			(at 133.35 142.24 0)
-			(hide yes)
-			(show_name no)
-			(do_not_autoplace no)
-			(effects
-				(font
-					(size 1.27 1.27)
-				)
-			)
-		)
-		(pin "1"
-		)
-		(pin "2"
-		)
-		(instances
-			(project "pcb"
-				(path "/bb6da232-368e-4a1f-bf9d-dbd7b03483b8"
-					(reference "J1")
-					(unit 1)
-				)
-			)
-		)
-	)
-	(symbol
 		(lib_id "seed studio xiao:XIAO-RP2350-SMD")
 		(at 137.16 109.22 0)
@@
 			)
 		)
-		(property "Value" "XIAO-RP2350-SMD-MODEL"
+		(property "Value" "XIAO-RP2350-SMD"
 			(at 139.3033 133.35 0)
 			(show_name no)
@@
 			)
 		)
-		(property "Footprint" "seed studio xiao:XIAO-RP2350-SMD-MODEL"
+		(property "Footprint" "Seeed_Studio_XIAO_Series:XIAO-RP2350-SMD"
 			(at 137.668 98.806 0)
 			(hide yes)
